File: PCB/Plonke.kicad_pcb (KiCad board)
At the start: 2 copper layers, 232 x 101 mm, 112 parts, among them J1 USB_C_Receptacle_USB2.0_16P, J2 AVR-ISP-6, SW1 SW_Push, SW10 SW_Push, SW11 SW_Push, SW12 SW_Push, SW13 SW_Push, SW14 SW_Push, SW15 SW_Push, SW16 SW_Push, SW17 SW_Push, SW18 SW_Push, SW19 SW_Push, SW2 SW_Push, SW20 SW_Push, SW21 SW_Push, SW22 SW_Push, SW23 SW_Push, SW24 SW_Push, SW25 SW_Push, SW26 SW_Push, SW27 SW_Push, SW28 SW_Push, SW29 SW_Push, SW3 SW_Push, SW30 SW_Push, SW31 SW_Push, SW32 SW_Push, SW33 SW_Push, SW34 SW_Push, SW35 SW_Push, SW36 SW_Push, SW37 SW_Push, SW38 SW_Push, SW39 SW_Push, SW4 SW_Push, SW40 SW_Push, SW41 SW_Push, SW42 SW_Push, SW43 SW_Push, SW44 SW_Push, SW45 SW_Push, SW46 SW_Push, SW47 SW_Push, SW5 SW_Push, SW6 SW_Push, SW7 SW_Push, SW8 SW_Push, SW9 SW_Push, U1 ATmega32U4-A, U2 USB6B1, Y1 Crystal_GND24_Small

Commit message: ok i'm going to finish this now
if going 4layer makes this easier i will do it. just one more layer bro, just one more....
Parts:
- moved U2 14.7 mm to (140.2, 49.5), turned to 180 degrees
- moved Y1 7.75 mm to (126.3, 49.8)
- moved D17 6.38 mm to (116.4, 56.0)
- moved D29 6.38 mm to (119.4, 61.0)
- moved D41 6.38 mm to (122.6, 66.0)
- moved D5 6.38 mm to (113.4, 51.0)
- moved D16 6.19 mm to (97.8, 56.0)
- moved D28 6.19 mm to (100.6, 61.0)
- moved D4 6.19 mm to (94.8, 51.0)
- moved D40 6.19 mm to (103.8, 66.0)
- moved R1 6.00 mm to (82.4, 54.4)
- moved R2 6.00 mm to (108.6, 61.6)
- moved D15 5.88 mm to (79.1, 56.0)
- moved D27 5.88 mm to (82.1, 61.0)
- moved D3 5.88 mm to (76.1, 51.0)
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Routing:
- net Net-(D38-A): track 150.0 -> 0.00 mm
- net GND: track 0.00 -> 125.7 mm
- net VBUS: track 0.00 -> 98.2 mm, vias 0 -> 1
- net Net-(D37-A): track 77.4 -> 0.00 mm
- net RESET: track 0.00 -> 71.9 mm, vias 0 -> 1
- net Net-(J1-CC2): track 0.00 -> 70.4 mm, vias 0 -> 1
- net Net-(D25-A): track 65.4 -> 0.00 mm
- net Net-(D13-A): track 53.9 -> 0.00 mm
- net Net-(U1-D-): track 0.00 -> 45.0 mm, vias 0 -> 1
- net Net-(J1-CC1): track 0.00 -> 43.3 mm, vias 0 -> 1
- net D+: track 0.00 -> 43.3 mm, vias 0 -> 1
- net Net-(D1-A): track 41.7 -> 0.00 mm
- net Net-(D6-A): track 39.5 -> 0.00 mm
- net C7: track 0.00 -> 39.1 mm
- net Net-(U1-XTAL2): track 0.00 -> 37.4 mm, vias 0 -> 1
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
Commit message: Spooky Commit
Hand Routed Traces
Parts:
- added ?: , , F.Cu at (54.8, 126.0)
- added ?: , , F.Cu at (226.2, 88.0)
- added ?: , , F.Cu at (226.2, 126.0)
- added REF**: MountingHole_3.2mm_M3, MountingHole:MountingHole_3.2mm_M3, F.Cu at (54.8, 88.0)
- D18, D19, D30, D31, D42, D6, D7: moved to F.Cu
- moved D42 70.7 mm to (123.9, 65.8)
- moved D30 55.5 mm to (122.3, 60.9)
- moved D31 54.0 mm to (175.1, 61.2)
- moved D18 42.3 mm to (120.9, 55.8)
- moved D19 40.1 mm to (176.8, 56.2)
- moved D6 33.1 mm to (119.3, 51.0)
- moved D7 30.8 mm to (178.6, 51.2)
- moved D43 17.5 mm to (188.8, 66.2)
- moved D32 16.2 mm to (190.6, 61.2)
- moved D20 15.0 mm to (192.4, 56.2)
- moved D44 14.2 mm to (204.3, 66.2)
- moved D8 13.8 mm to (194.2, 51.2)
- moved D41 13.3 mm to (109.3, 66.0)
- moved D33 12.9 mm to (206.1, 61.2)
- moved R2 12.1 mm to (96.5, 62.2), turned to 110 degrees
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Routing:
- net Net-(D42-A): track 0.00 -> 111.6 mm, vias 0 -> 1
- net Net-(D41-A): track 0.00 -> 97.0 mm
- net Net-(D30-A): track 0.00 -> 94.6 mm, vias 0 -> 1
- net Net-(D40-A): track 0.00 -> 93.7 mm, vias 0 -> 1
- net Net-(D39-A): track 0.00 -> 90.6 mm
- net Net-(D38-A): track 0.00 -> 89.0 mm
- net Net-(D37-A): track 0.00 -> 85.1 mm
- net Net-(D29-A): track 0.00 -> 85.0 mm, vias 0 -> 1
- net R1: track 0.00 -> 83.2 mm
- net Net-(D28-A): track 0.00 -> 81.1 mm, vias 0 -> 1
- net R3: track 0.00 -> 80.6 mm, vias 0 -> 1
- net R2: track 0.00 -> 80.1 mm
- net R4: track 0.00 -> 79.6 mm, vias 0 -> 1
- net Net-(D18-A): track 0.00 -> 79.6 mm, vias 0 -> 1
- net Net-(D27-A): track 0.00 -> 76.8 mm
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
Commit message: Take a gander
nearly there...
Parts:
- moved D12 15.9 mm to (250.8, 66.2)
- moved D47 15.9 mm to (256.2, 51.2)
- moved D11 15.9 mm to (235.3, 66.2)
- moved D46 15.9 mm to (240.7, 51.2)
- moved D43 15.9 mm to (194.2, 51.2)
- moved D8 15.9 mm to (188.8, 66.2)
- moved D44 15.9 mm to (209.7, 51.2)
- moved D9 15.9 mm to (204.3, 66.2)
- moved D10 15.9 mm to (219.8, 66.2)
- moved D45 15.9 mm to (225.2, 51.2)
- moved D31 10.6 mm to (178.6, 51.2)
- moved D7 10.6 mm to (175.1, 61.2)
- moved D20 5.32 mm to (190.6, 61.2)
- moved D32 5.32 mm to (192.4, 56.2)
- moved D21 5.32 mm to (206.1, 61.2)
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Routing:
- net Net-(D43-A): track 0.00 -> 96.8 mm
- net Net-(D44-A): track 0.00 -> 92.1 mm
- net Net-(D45-A): track 0.00 -> 90.6 mm
- net Net-(D46-A): track 0.00 -> 89.2 mm
- net Net-(D47-A): track 0.00 -> 88.7 mm
- net Net-(D34-A): track 0.00 -> 68.7 mm
- net Net-(D33-A): track 0.00 -> 67.3 mm
- net Net-(D35-A): track 0.00 -> 64.9 mm
- net Net-(D36-A): track 7.61 -> 64.7 mm
- net Net-(D21-A): track 0.00 -> 42.5 mm
- net Net-(D22-A): track 0.00 -> 42.1 mm
- net Net-(D23-A): track 0.00 -> 39.6 mm
- net Net-(D24-A): track 12.6 -> 40.8 mm
- net Net-(J1-CC2): track 52.8 -> 78.1 mm
- net GND: track 99.5 -> 118.2 mm
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
Commit message: Rows+Col Wired
now comes the worst part
Routing:
- net R1: track 83.2 -> 173.3 mm, vias 0 -> 2
- net R3: track 80.6 -> 168.2 mm, vias 1 -> 2
- net Net-(D31-A): track 0.00 -> 80.2 mm
- net R4: track 79.6 -> 150.5 mm
- net R2: track 80.1 -> 149.4 mm, vias 0 -> 1
- net Net-(D32-A): track 0.00 -> 68.8 mm, vias 0 -> 1
- net Net-(D19-A): track 0.00 -> 53.8 mm, vias 0 -> 1
- net Net-(D20-A): track 0.00 -> 45.6 mm
- net Net-(D7-A): track 0.00 -> 26.4 mm, vias 0 -> 1
- net Net-(D8-A): track 0.00 -> 19.2 mm

Commit message: final update for the night
Parts:
- J1: footprint Connector_USB:USB_C_Receptacle_Amphenol_12401548E4-2A -> Connector_USB:USB_C_Receptacle_XKB_U262-16XN-4BVC11
Connections:
- U1 pad 25: unconnected-(U1-PD4-Pad25) -> R1
- U1 pad 26: unconnected-(U1-PD6-Pad26) -> R2
- U1 pad 27: unconnected-(U1-PD7-Pad27) -> R3
- U1 pad 28: unconnected-(U1-PB4-Pad28) -> R4
Routing:
- net R1: track 173.3 -> 188.2 mm
- net GND: track 118.2 -> 106.5 mm
- net R2: track 149.4 -> 161.0 mm
- net R4: track 150.5 -> 161.2 mm
- net R3: track 168.2 -> 178.4 mm
- net Net-(J1-CC2): track 78.1 -> 85.1 mm, vias 1 -> 2
- net Net-(J1-D--PadA7): track 14.6 -> 16.0 mm

Commit message: WIRING DONE
lfg
Parts:
- moved ? 19.0 mm to (245.2, 88.0)
- moved ? 19.0 mm to (245.2, 126.0)
Connections:
- U1 pad 1: unconnected-(U1-PE6-Pad1) -> C9
- U1 pad 29: unconnected-(U1-PB5-Pad29) -> C6
- U1 pad 30: unconnected-(U1-PB6-Pad30) -> C5
- U1 pad 31: unconnected-(U1-PC6-Pad31) -> C4
- U1 pad 32: unconnected-(U1-PC7-Pad32) -> C3
- U1 pad 33: unconnected-(U1-~{HWB}/PE2-Pad33) -> C2
- U1 pad 36: unconnected-(U1-PF7-Pad36) -> C1
- U1 pad 37: unconnected-(U1-PF6-Pad37) -> C7
- U1 pad 38: unconnected-(U1-PF5-Pad38) -> C8
- U1 pad 39: unconnected-(U1-PF4-Pad39) -> C12
- U1 pad 40: unconnected-(U1-PF1-Pad40) -> C11
- U1 pad 41: unconnected-(U1-PF0-Pad41) -> C10
Routing:
- net C1: track 57.7 -> 211.2 mm, vias 0 -> 5
- net C2: track 57.8 -> 192.6 mm, vias 0 -> 5
- net C12: track 58.0 -> 187.9 mm, vias 0 -> 3
- net C3: track 56.7 -> 173.7 mm, vias 0 -> 5
- net C11: track 57.9 -> 167.0 mm, vias 0 -> 3
- net C10: track 58.0 -> 145.0 mm, vias 0 -> 3
- net C4: track 57.8 -> 138.2 mm, vias 0 -> 3
- net C8: track 57.8 -> 134.2 mm, vias 0 -> 1
- net C9: track 58.0 -> 120.2 mm, vias 0 -> 3
- net C5: track 57.8 -> 118.0 mm, vias 0 -> 3
- net C7: track 39.1 -> 73.4 mm, vias 0 -> 1
- net C6: track 60.8 -> 90.1 mm, vias 0 -> 1
- net Net-(D34-A): track 68.7 -> 65.8 mm
- net Net-(D25-A): track 71.2 -> 74.0 mm
- net Net-(D35-A): track 64.9 -> 67.7 mm
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Other:
- board text added: "hello from aotearoa"
- board text added: "the plonke"
