File: PCB/Plonke.kicad_pcb (KiCad board)
At the start: 2 copper layers, 232 x 101 mm, 116 parts, among them J1 USB_C_Receptacle_USB2.0_16P, J2 AVR-ISP-6, SW1 SW_Push, SW10 SW_Push, SW11 SW_Push, SW12 SW_Push, SW13 SW_Push, SW14 SW_Push, SW15 SW_Push, SW16 SW_Push, SW17 SW_Push, SW18 SW_Push, SW19 SW_Push, SW2 SW_Push, SW20 SW_Push, SW21 SW_Push, SW22 SW_Push, SW23 SW_Push, SW24 SW_Push, SW25 SW_Push, SW26 SW_Push, SW27 SW_Push, SW28 SW_Push, SW29 SW_Push, SW3 SW_Push, SW30 SW_Push, SW31 SW_Push, SW32 SW_Push, SW33 SW_Push, SW34 SW_Push, SW35 SW_Push, SW36 SW_Push, SW37 SW_Push, SW38 SW_Push, SW39 SW_Push, SW4 SW_Push, SW40 SW_Push, SW41 SW_Push, SW42 SW_Push, SW43 SW_Push, SW44 SW_Push, SW45 SW_Push, SW46 SW_Push, SW47 SW_Push, SW5 SW_Push, SW6 SW_Push, SW7 SW_Push, SW8 SW_Push, SW9 SW_Push, U1 ATmega32U4-A, U2 USB6B1, Y1 Crystal_GND24_Small

Commit message: ok actually finally wired now
i forgot to connect the col's together
classic mistake but with some creative wiring i got there eventually.
Routing:
- net R4: track 161.2 -> 251.8 mm, vias 1 -> 3
- net R1: track 188.2 -> 270.7 mm, vias 2 -> 4
- net R2: track 161.0 -> 241.4 mm, vias 1 -> 5
- net R3: track 178.4 -> 249.5 mm, vias 2 -> 4
- net Net-(J1-CC2): track 85.1 -> 86.0 mm

Commit message: chop and change
needs drc next
Routing:
- net GND: track 106.5 -> 113.3 mm, vias 0 -> 1
- net C8: track 134.2 -> 130.5 mm
- net C1: track 211.5 -> 208.1 mm
- net C4: track 138.1 -> 136.6 mm

Commit message: i have no idea what i'm doing
please help me (drc)
why must you hate my diode footprints i don't know what i'm doing plea s leav me aloneeeeeeee
Parts:
- moved R5 1.34 mm to (201.3, 61.0)
Routing:
- net R2: track 241.4 -> 245.2 mm, vias 5 -> 4
- net GND: track 113.3 -> 116.5 mm
- net VBUS: track 101.1 -> 103.7 mm
- net Net-(J1-CC2): track 86.0 -> 83.9 mm
- net Net-(D3-A): track 47.0 -> 48.5 mm
- net Net-(D43-A): track 96.8 -> 97.3 mm
