File: PCB/Plonke.kicad_sch (KiCad schematic)
At the start: 17 parts, among them J1 USB_C_Receptacle_USB2.0_16P, J2 AVR-ISP-6, U1 ATmega32U4-A, U2 USB6B1, Y1 Crystal_GND24_Small

Commit message: ok i'm going to finish this now
if going 4layer makes this easier i will do it. just one more layer bro, just one more....
Parts:
- J1: footprint Connector_USB:USB_C_Receptacle_Amphenol_12401548E4-2A -> Connector_USB:USB_C_Receptacle_XKB_U262-16XN-4BVC11
Changed lines of the file:
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@@
 			)
 		)
-		(property "Footprint" "Connector_USB:USB_C_Receptacle_Amphenol_12401548E4-2A"
+		(property "Footprint" "Connector_USB:USB_C_Receptacle_XKB_U262-16XN-4BVC11"
 			(at 38.1 41.91 0)
 			(effects
@@
 		)
 		(instances
-			(project "Ricky_Keyboard"
+			(project "Plonke"
 				(path "/8b9b9087-ba2f-4a40-b105-221ef5fe39ca"
 					(page "2")

Commit message: final update for the night
Connections:
- net R1: now reaches U1.25 (PD4)
- net R2: now reaches U1.26 (PD6)
- net R3: now reaches U1.27 (PD7)
- net R4: now reaches U1.28 (PB4)
Changed lines of the file:
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@@
+	(wire
+		(pts
+			(xy 219.71 54.61) (xy 228.6 54.61)
+		)
+		(stroke
+			(width 0)
+			(type default)
+		)
+	)
 	(wire
 		(pts
@@
 	(wire
 		(pts
-			(xy 181.61 80.01) (xy 181.61 77.47)
+			(xy 219.71 90.17) (xy 228.6 90.17)
 		)
 		(stroke
@@
 	(wire
 		(pts
-			(xy 179.07 49.53) (xy 189.23 49.53)
+			(xy 181.61 80.01) (xy 181.61 77.47)
 		)
 		(stroke
@@
 	(wire
 		(pts
-			(xy 49.53 45.72) (xy 64.77 45.72)
+			(xy 179.07 49.53) (xy 189.23 49.53)
 		)
 		(stroke
@@
 	(wire
 		(pts
-			(xy 179.07 54.61) (xy 189.23 54.61)
+			(xy 49.53 45.72) (xy 64.77 45.72)
 		)
 		(stroke
@@
 	(wire
 		(pts
-			(xy 49.53 40.64) (xy 64.77 40.64)
+			(xy 219.71 92.71) (xy 228.6 92.71)
 		)
 		(stroke
@@
 	(wire
 		(pts
-			(xy 162.56 52.07) (xy 168.91 52.07)
+			(xy 179.07 54.61) (xy 189.23 54.61)
 		)
 		(stroke
@@
 	(wire
 		(pts
-			(xy 181.61 77.47) (xy 189.23 77.47)
+			(xy 49.53 40.64) (xy 64.77 40.64)
 		)
 		(stroke
@@
 	(wire
 		(pts
-			(xy 49.53 40.64) (xy 49.53 41.91)
+			(xy 162.56 52.07) (xy 168.91 52.07)
 		)
 		(stroke
@@
 	(wire
 		(pts
-			(xy 176.53 52.07) (xy 168.91 52.07)
+			(xy 181.61 77.47) (xy 189.23 77.47)
 		)
 		(stroke
@@
 	(wire
 		(pts
-			(xy 176.53 54.61) (xy 179.07 54.61)
+			(xy 49.53 40.64) (xy 49.53 41.91)
 		)
 		(stroke
@@
 	(wire
 		(pts
-			(xy 57.15 33.02) (xy 59.69 33.02)
+			(xy 176.53 52.07) (xy 168.91 52.07)
 		)
 		(stroke
@@
 	(wire
 		(pts
-			(xy 181.61 52.07) (xy 184.15 52.07)
+			(xy 176.53 54.61) (xy 179.07 54.61)
 		)
 		(stroke
@@
 	(wire
 		(pts
-			(xy 168.91 49.53) (xy 168.91 52.07)
+			(xy 57.15 33.02) (xy 59.69 33.02)
 		)
 		(stroke
@@
 	(wire
 		(pts
-			(xy 185.42 69.85) (xy 189.23 69.85)
+			(xy 181.61 52.07) (xy 184.15 52.07)
 		)
 		(stroke
@@
 	(wire
 		(pts
-			(xy 181.61 35.56) (xy 181.61 36.83)
+			(xy 168.91 49.53) (xy 168.91 52.07)
 		)
 		(stroke
@@
 	(wire
 		(pts
-			(xy 57.15 33.02) (xy 57.15 34.29)
+			(xy 219.71 85.09) (xy 228.6 85.09)
 		)
 		(stroke
@@
 	(wire
 		(pts
-			(xy 181.61 44.45) (xy 189.23 44.45)
+			(xy 185.42 69.85) (xy 189.23 69.85)
 		)
 		(stroke
@@
 	(wire
 		(pts
-			(xy 57.15 31.75) (xy 57.15 33.02)
+			(xy 181.61 35.56) (xy 181.61 36.83)
 		)
 		(stroke
@@
 	(wire
 		(pts
-			(xy 168.91 52.07) (xy 168.91 54.61)
+			(xy 57.15 33.02) (xy 57.15 34.29)
 		)
 		(stroke
@@
 	(wire
 		(pts
-			(xy 49.53 39.37) (xy 49.53 40.64)
+			(xy 181.61 44.45) (xy 189.23 44.45)
 		)
 		(stroke
@@
 	(wire
 		(pts
-			(xy 207.01 35.56) (xy 204.47 35.56)
+			(xy 57.15 31.75) (xy 57.15 33.02)
 		)
 		(stroke
@@
 	(wire
 		(pts
-			(xy 201.93 35.56) (xy 204.47 35.56)
+			(xy 168.91 52.07) (xy 168.91 54.61)
 		)
 		(stroke
@@
 	(wire
 		(pts
-			(xy 201.93 36.83) (xy 201.93 35.56)
+			(xy 49.53 39.37) (xy 49.53 40.64)
 		)
 		(stroke
@@
 		)
 	)
+	(wire
+		(pts
+			(xy 207.01 35.56) (xy 204.47 35.56)
+		)
+		(stroke
+			(width 0)
+			(type default)
+		)
+	)
+	(wire
+		(pts
+			(xy 201.93 35.56) (xy 204.47 35.56)
+		)
+		(stroke
+			(width 0)
+			(type default)
+		)
+	)
+	(wire
+		(pts
+			(xy 201.93 36.83) (xy 201.93 35.56)
+		)
+		(stroke
+			(width 0)
+			(type default)
+		)
+	)
 	(global_label "MOSI"
 		(shape input)
@@
 		)
 	)
+	(global_label "R1"
+		(shape input)
+		(at 228.6 85.09 0)
+		(fields_autoplaced yes)
+		(effects
+			(font
+				(size 1.27 1.27)
+			)
+			(justify left)
+		)
+		(property "Intersheetrefs" "${INTERSHEET_REFS}"
+			(at 234.0647 85.09 0)
+			(effects
+				(font
+					(size 1.27 1.27)
+				)
+				(justify left)
+				(hide yes)
+			)
+		)
+	)
 	(global_label "SCL"
 		(shape input)
@@
 		)
 	)
+	(global_label "R2"
+		(shape input)
+		(at 228.6 90.17 0)
+		(fields_autoplaced yes)
+		(effects
+			(font
+				(size 1.27 1.27)
+			)
+			(justify left)
+		)
+		(property "Intersheetrefs" "${INTERSHEET_REFS}"
+			(at 234.0647 90.17 0)
+			(effects
+				(font
+					(size 1.27 1.27)
+				)
+				(justify left)
+				(hide yes)
+			)
+		)
+	)
 	(global_label "VBUS"
 		(shape input)
@@
 		)
 	)
+	(global_label "R4"
+		(shape input)
+		(at 228.6 54.61 0)
+		(fields_autoplaced yes)
+		(effects
+			(font
+				(size 1.27 1.27)
+			)
+			(justify left)
+		)
+		(property "Intersheetrefs" "${INTERSHEET_REFS}"
+			(at 234.0647 54.61 0)
+			(effects
+				(font
+					(size 1.27 1.27)
+				)
+				(justify left)
+				(hide yes)
+			)
+		)
+	)
+	(global_label "R3"
+		(shape input)
+		(at 228.6 92.71 0)
+		(fields_autoplaced yes)
+		(effects
+			(font
+				(size 1.27 1.27)
+			)
+			(justify left)
+		)
+		(property "Intersheetrefs" "${INTERSHEET_REFS}"
+			(at 234.0647 92.71 0)
+			(effects
+				(font
+					(size 1.27 1.27)
+				)
+				(justify left)
+				(hide yes)
+			)
+		)
+	)
 	(global_label "SCL"
 		(shape input)
@@
 	(sheet
 		(at 80.01 109.22)
-		(size 12.7 3.81)
+		(size 24.13 16.51)
 		(fields_autoplaced yes)
 		(stroke
@@
 		)
 		(property "Sheetfile" "sheetMatrix.kicad_sch"
-			(at 80.01 113.6146 0)
-			(effects
-				(font
+			(at 80.01 126.3146 0)
+			(effects
+				(font

Commit message: WIRING DONE
lfg
Connections:
- net C9: now reaches U1.1 (PE6)
- net C6: now reaches U1.29 (PB5)
- net C5: now reaches U1.30 (PB6)
- net C4: now reaches U1.31 (PC6)
- net C3: now reaches U1.32 (PC7)
- net C2: now reaches U1.33 (~{HWB}/PE2)
- net C1: now reaches U1.36 (PF7)
- net C7: now reaches U1.37 (PF6)
- net C8: now reaches U1.38 (PF5)
- net C12: now reaches U1.39 (PF4)
- net C11: now reaches U1.40 (PF1)
- net C10: now reaches U1.41 (PF0)
